File: P15pwr.kicad_sch (KiCad schematic)
At the start: 9 parts, among them U5 L78M12

Commit message: upgrade to Kicad 9
Parts:
- C15: JLCPCB C696814 -> (none); LCSC Part # (none) -> C696814
- C26: JLCPCB C12891 -> (none); LCSC Part # (none) -> C12891
- C27: JLCPCB C50254 -> (none); LCSC Part # (none) -> C50254
- D1: JLCPCB C60396 -> (none); LCSC Part # (none) -> C60396
- R89: JLCPCB C31850 -> (none); LCSC Part # (none) -> C31850
- R90: JLCPCB C25804 -> (none); LCSC Part # (none) -> C25804
- U5: JLCPCB C22357875 -> (none); LCSC Part # (none) -> C22357875
Changed lines of the file:
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@@
 			)
 		)
-		(property "JLCPCB" "C60396"
+		(property "LCSC Part #" "C60396"
 			(at 44.45 44.45 0)
 			(effects
@@
 			)
 		)
-		(property "JLCPCB" "C22357875"
+		(property "LCSC Part #" "C22357875"
 			(at 110.49 44.45 0)
 			(effects
@@
 			)
 		)
-		(property "JLCPCB" "C50254"
+		(property "LCSC Part #" "C50254"
 			(at 95.25 53.34 0)
 			(effects
@@
 			)
 		)
-		(property "JLCPCB" "C31850"
+		(property "LCSC Part #" "C31850"
 			(at 85.09 49.53 0)
 			(effects
@@
 			)
 		)
-		(property "JLCPCB" "C25804"
+		(property "LCSC Part #" "C25804"
 			(at 147.32 49.53 0)
 			(effects
@@
 			)
 		)
-		(property "JLCPCB" "C696814"
+		(property "LCSC Part #" "C696814"
 			(at 57.15 53.34 0)
 			(effects
@@
 			)
 		)
-		(property "JLCPCB" "C12891"
+		(property "LCSC Part #" "C12891"
 			(at 127 53.34 0)
 			(effects
