File: P15slt.kicad_sch (KiCad schematic)
At the start: 27 parts, among them J1 Screw_Terminal_01x02, J3 Slot: Booster, J4 Slot-a1, J5 Barrel_Jack_Switch, J6 Screw_Terminal_01x04, J7 Slot: Master, Q1 BC847

Commit message: upgrade to Kicad 9
Parts:
- D2, D3: JLCPCB C60396 -> (none); LCSC Part # (none) -> C60396
- Q1: JLCPCB C7420337 -> (none); LCSC Part # (none) -> C7420337
- R1, R2: JLCPCB C17901 -> (none); LCSC Part # (none) -> C17901
- R3: JLCPCB C23212 -> (none); LCSC Part # (none) -> C23212
- R4: JLCPCB C13167 -> (none); LCSC Part # (none) -> C13167
Changed lines of the file:
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@@
 			)
 		)
-		(property "JLCPCB" "C60396"
+		(property "LCSC Part #" "C60396"
 			(at 238.76 53.34 0)
 			(effects
@@
 			)
 		)
-		(property "JLCPCB" "C17901"
+		(property "LCSC Part #" "C17901"
 			(at 193.04 59.69 90)
 			(effects
@@
 			)
 		)
-		(property "JLCPCB" "C60396"
+		(property "LCSC Part #" "C60396"
 			(at 238.76 57.15 0)
 			(effects
@@
 			)
 		)
-		(property "JLCPCB" "C17901"
+		(property "LCSC Part #" "C17901"
 			(at 193.04 57.15 90)
 			(effects
@@
 			)
 		)
-		(property "JLCPCB" "C7420337"
+		(property "LCSC Part #" "C7420337"
 			(at 223.52 66.04 0)
 			(effects
@@
 			)
 		)
-		(property "JLCPCB" "C23212"
+		(property "LCSC Part #" "C23212"
 			(at 218.44 60.96 90)
 			(effects
@@
 			)
 		)
-		(property "JLCPCB" "C13167"
+		(property "LCSC Part #" "C13167"
 			(at 238.76 60.96 90)
 			(effects
